File: hardware/rev0/ram_section.sch (KiCad schematic (older format))
At the start: 2 parts, among them IC1 ECP5-BGA256, U10 S27KS0641

Commit message: hardware: add part numbers
Parts:
- U10: Description (none) -> IC DRAM 64M PARALLEL 24BGA; Manufacturer_Name (none) -> Cypress Semiconductor; Manufacturer_Part_Number (none) -> S27KS0641DPBHI020
Changed lines of the file:
@@
 EESchema Schematic File Version 4
-LIBS:luna_rev0-cache
 EELAYER 30 0
 EELAYER END
@@
 F 3 "" H 5400 3950 50  0001 C CNN
 F 4 "ANY" H 5400 4850 50  0001 C CNN "Source"
+F 5 "IC DRAM 64M PARALLEL 24BGA" H 5400 4850 50  0001 C CNN "Description"
+F 6 "Cypress Semiconductor" H 5400 4850 50  0001 C CNN "Manufacturer_Name"
+F 7 "S27KS0641DPBHI020" H 5400 4850 50  0001 C CNN "Manufacturer_Part_Number"
 	1    5400 4850
 	-1   0    0    -1

Commit message: hardware: normalize BOM fields
make compatible with kicad-bom-scripts
Parts:
- IC1: Height 1.7 -> (none); Manufacturer (none) -> Lattice; Manufacturer_Name Lattice -> (none); Manufacturer_Part_Number LFE5U-12F-6BG256C -> (none); Mouser Part Number 842-LFE5U12F6BG256C -> (none); Mouser Price/Stock https://www.mouser.com/Search/Refine.aspx?Keyword=842-LFE5U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 -> (none); Part Number (none) -> LFE5U-12F-6BG256C
- U10: Manufacturer (none) -> Cypress Semiconductor; Manufacturer_Name Cypress Semiconductor -> (none); Manufacturer_Part_Number S27KS0641DPBHI020 -> (none); Part Number (none) -> S27KS0641DPBHI020; Source ANY -> (none)
Changed lines of the file:
@@
 F 3 "" H -2000 6500 50  0001 L CNN
 F 4 "FPGA - Field Programmable Gate Array ECP5; 12k LUTs; 1.1V" H -2000 6400 50  0001 L CNN "Description"
-F 5 "1.7" H -2000 6750 50  0001 L CNN "Height"
-F 6 "Lattice" H -1950 7350 50  0001 L CNN "Manufacturer_Name"
-F 7 "LFE5U-12F-6BG256C" H -1950 7250 50  0001 L CNN "Manufacturer_Part_Number"
-F 8 "842-LFE5U12F6BG256C" H -1300 5950 50  0001 L CNN "Mouser Part Number"
-F 9 "https://www.mouser.com/Search/Refine.aspx?Keyword=842-LFE5U12F6BG256C" H -1650 5800 50  0001 L CNN "Mouser Price/Stock"
+F 5 "Lattice" H -1950 7350 50  0001 L CNN "Manufacturer"
+F 6 "LFE5U-12F-6BG256C" H -1950 7250 50  0001 L CNN "Part Number"
 	3    1650 2100
 	1    0    0    -1
@@
 F 2 "luna:BGA-24_5x5_6.0x8.0mm" H 6000 3950 50  0001 C CNN
 F 3 "" H 5400 3950 50  0001 C CNN
-F 4 "ANY" H 5400 4850 50  0001 C CNN "Source"
-F 5 "IC DRAM 64M PARALLEL 24BGA" H 5400 4850 50  0001 C CNN "Description"
-F 6 "Cypress Semiconductor" H 5400 4850 50  0001 C CNN "Manufacturer_Name"
-F 7 "S27KS0641DPBHI020" H 5400 4850 50  0001 C CNN "Manufacturer_Part_Number"
+F 4 "IC DRAM 64M PARALLEL 24BGA" H 5400 4850 50  0001 C CNN "Description"
+F 5 "Cypress Semiconductor" H 5400 4850 50  0001 C CNN "Manufacturer"
+F 6 "S27KS0641DPBHI020" H 5400 4850 50  0001 C CNN "Part Number"
 	1    5400 4850
 	-1   0    0    -1
