File: hardware/rev0/right_side_indicators.sch (KiCad schematic (older format))
At the start: 1 part, among them IC1 ECP5-BGA256

Commit message: hardware: normalize BOM fields
make compatible with kicad-bom-scripts
Parts:
- IC1: Height 1.7 -> (none); Manufacturer (none) -> Lattice; Manufacturer_Name Lattice -> (none); Manufacturer_Part_Number LFE5U-12F-6BG256C -> (none); Mouser Part Number 842-LFE5U12F6BG256C -> (none); Mouser Price/Stock https://www.mouser.com/Search/Refine.aspx?Keyword=842-LFE5U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 -> (none); Part Number (none) -> LFE5U-12F-6BG256C
Changed lines of the file:
@@
 F 3 "" H -1500 6400 50  0001 L CNN
 F 4 "FPGA - Field Programmable Gate Array ECP5; 12k LUTs; 1.1V" H -1500 6300 50  0001 L CNN "Description"
-F 5 "1.7" H -1500 6650 50  0001 L CNN "Height"
-F 6 "Lattice" H -1450 7250 50  0001 L CNN "Manufacturer_Name"
-F 7 "LFE5U-12F-6BG256C" H -1450 7150 50  0001 L CNN "Manufacturer_Part_Number"
-F 8 "842-LFE5U12F6BG256C" H -800 5850 50  0001 L CNN "Mouser Part Number"
-F 9 "https://www.mouser.com/Search/Refine.aspx?Keyword=842-LFE5U12F6BG256C" H -1150 5700 50  0001 L CNN "Mouser Price/Stock"
+F 5 "Lattice" H -1450 7250 50  0001 L CNN "Manufacturer"
+F 6 "LFE5U-12F-6BG256C" H -1450 7150 50  0001 L CNN "Part Number"
 	5    2150 2000
 	1    0    0    -1
