File: hardware/rev0/luna_rev0.kicad_pcb (KiCad board)
At the start: 4 copper layers, 48.9 x 50 mm, 132 parts, among them IC1 ECP5-BGA256, J1 USB_B_Micro, J2 USB_B_Micro, J3 USB_A, J4 USB_B_Micro, J5 Conn_ARM_JTAG_SWD_10, J6 Conn_ARM_JTAG_SWD_10, J7 Conn_02x02_Counter_Clockwise, J8 Conn_Coaxial, J9 Conn_Coaxial, SW1 BTN_RECOVERY, SW2 BTN_DFU, SW3 BTN_RESET, U1 AP22814-SOT, U10 S27KS0641, U11 USB3343, U12 AP22814-SOT, U2 MIC5504-1.8YM5, U3 MIC5219-3.3YM5, U4 TCR2EE11, U5 MIC5504-2.5YM5, U6 ATSAMD21G18A-AUT, U7 W25Q32JVSS, U8 USB3343, U9 USB3343, Y1 DSC60xx

Commit message: hardware: correct TCR2EE11 symbol pin numbering
Parts:
- C10, C11, C12, C13, C14, C15, C16, C17, C18, C23, C24, C25, C26, C7, C8, C9: value 0.1u -> 0.1uF
Connections:
- U4 pad 5: (no net) -> Net-(U4-Pad5)
Changed lines of the file:
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@@
     (zones 0)
     (modules 132)
-    (nets 284)
+    (nets 285)
   )
   (page A4)
@@
   (net 282 /DEBUG_SPI_CS)
   (net 283 "Net-(IC1-PadP12)")
+  (net 284 "Net-(U4-Pad5)")
   (net_class Default "This is the default net class."
     (clearance 0.127)
@@
     (add_net "Net-(U11-Pad20)")
     (add_net "Net-(U2-Pad4)")
+    (add_net "Net-(U4-Pad5)")
     (add_net "Net-(U5-Pad4)")
     (add_net "Net-(U6-Pad32)")
@@
       (effects (font (size 1 1) (thickness 0.15)) (justify mirror))
     )
-    (fp_text value 0.1u (at 0 -1.17 90) (layer B.Fab)
+    (fp_text value 0.1uF (at 0 -1.17 90) (layer B.Fab)
       (effects (font (size 1 1) (thickness 0.15)) (justify mirror))
     )
@@
       (effects (font (size 1 1) (thickness 0.15)) (justify mirror))
     )
-    (fp_text value 0.1u (at 0 -1.17) (layer B.Fab)
+    (fp_text value 0.1uF (at 0 -1.17) (layer B.Fab)
       (effects (font (size 1 1) (thickness 0.15)) (justify mirror))
     )
@@
       (effects (font (size 1 1) (thickness 0.15)) (justify mirror))
     )
-    (fp_text value 0.1u (at 0 -1.17) (layer B.Fab)
+    (fp_text value 0.1uF (at 0 -1.17) (layer B.Fab)
       (effects (font (size 1 1) (thickness 0.15)) (justify mirror))
     )
@@
       (effects (font (size 1 1) (thickness 0.15)) (justify mirror))
     )
-    (fp_text value 0.1u (at 0 -1.17) (layer B.Fab)
+    (fp_text value 0.1uF (at 0 -1.17) (layer B.Fab)
       (effects (font (size 1 1) (thickness 0.15)) (justify mirror))
     )
@@
       (effects (font (size 1 1) (thickness 0.15)) (justify mirror))
     )
-    (fp_text value 0.1u (at 0 -1.17) (layer B.Fab)
+    (fp_text value 0.1uF (at 0 -1.17) (layer B.Fab)
       (effects (font (size 1 1) (thickness 0.15)) (justify mirror))
     )
@@
       (effects (font (size 1 1) (thickness 0.15)) (justify mirror))
     )
-    (fp_text value 0.1u (at 0 -1.17) (layer B.Fab)
+    (fp_text value 0.1uF (at 0 -1.17) (layer B.Fab)
       (effects (font (size 1 1) (thickness 0.15)) (justify mirror))
     )
@@
       (effects (font (size 1 1) (thickness 0.15)) (justify mirror))
     )
-    (fp_text value 0.1u (at 0 -1.17 90) (layer B.Fab)
+    (fp_text value 0.1uF (at 0 -1.17 90) (layer B.Fab)
       (effects (font (size 1 1) (thickness 0.15)) (justify mirror))
     )
@@
       (effects (font (size 1 1) (thickness 0.15)))
     )
-    (fp_text value 0.1u (at 0 1.17 270) (layer F.Fab)
+    (fp_text value 0.1uF (at 0 1.17 270) (layer F.Fab)
       (effects (font (size 1 1) (thickness 0.15)))
     )
@@
       (effects (font (size 1 1) (thickness 0.15)) (justify mirror))
     )
-    (fp_text value 0.1u (at 0 -1.17 90) (layer B.Fab)
+    (fp_text value 0.1uF (at 0 -1.17 90) (layer B.Fab)
       (effects (font (size 1 1) (thickness 0.15)) (justify mirror))
     )
@@
       (effects (font (size 1 1) (thickness 0.15)))
     )
-    (fp_text value 0.1u (at 0 1.17 90) (layer F.Fab)
+    (fp_text value 0.1uF (at 0 1.17 90) (layer F.Fab)
       (effects (font (size 1 1) (thickness 0.15)))
     )
@@
       (effects (font (size 1 1) (thickness 0.15)) (justify mirror))
     )
-    (fp_text value 0.1u (at 0 -1.17 90) (layer B.Fab)
+    (fp_text value 0.1uF (at 0 -1.17 90) (layer B.Fab)
       (effects (font (size 1 1) (thickness 0.15)) (justify mirror))
     )
@@
       (effects (font (size 1 1) (thickness 0.15)))
     )
-    (fp_text value 0.1u (at 0 1.17) (layer F.Fab)
+    (fp_text value 0.1uF (at 0 1.17) (layer F.Fab)
       (effects (font (size 1 1) (thickness 0.15)))
     )
@@
       (effects (font (size 1 1) (thickness 0.15)) (justify mirror))
     )
-    (fp_text value 0.1u (at 0 -1.17) (layer B.Fab)
+    (fp_text value 0.1uF (at 0 -1.17) (layer B.Fab)
       (effects (font (size 1 1) (thickness 0.15)) (justify mirror))
     )
@@
       (effects (font (size 1 1) (thickness 0.15)) (justify mirror))
     )
-    (fp_text value 0.1u (at 0 -1.17 90) (layer B.Fab)
+    (fp_text value 0.1uF (at 0 -1.17 90) (layer B.Fab)
       (effects (font (size 1 1) (thickness 0.15)) (justify mirror))
     )
@@
       (effects (font (size 1 1) (thickness 0.15)) (justify mirror))
     )
-    (fp_text value 0.1u (at 0 -1.17 90) (layer B.Fab)
+    (fp_text value 0.1uF (at 0 -1.17 90) (layer B.Fab)
       (effects (font (size 1 1) (thickness 0.15)) (justify mirror))
     )
@@
       (effects (font (size 1 1) (thickness 0.15)) (justify mirror))
     )
-    (fp_text value 0.1u (at 0 -1.17) (layer B.Fab)
+    (fp_text value 0.1uF (at 0 -1.17) (layer B.Fab)
       (effects (font (size 1 1) (thickness 0.15)) (justify mirror))
     )
@@
     (pad 3 smd rect (at -0.7 0.5) (size 0.45 0.3) (layers F.Cu F.Paste F.Mask)
       (net 5 +2V5))
-    (pad 5 smd rect (at 0.7 -0.5) (size 0.45 0.3) (layers F.Cu F.Paste F.Mask))
+    (pad 5 smd rect (at 0.7 -0.5) (size 0.45 0.3) (layers F.Cu F.Paste F.Mask)
+      (net 284 "Net-(U4-Pad5)"))
     (pad 2 smd rect (at -0.7 0) (size 0.45 0.3) (layers F.Cu F.Paste F.Mask)
       (net 2 GND))
